File: kicad-files/Cap Touch Controller.sch (KiCad schematic (older format))
At the start: 28 parts, among them J1 USB_C_Receptacle_USB2.0, J2 8-pin_header, J3 8-pin_header, U1 ATSAMD21J15B-A, U2 MIC5365-2.8YC5

Commit message: New Files
Connections:
- net labels removed: LED_1, LED_2, LED_3, LED_4, LED_A, LED_B
- wire segments 41 -> 20
Other:
- moved on the sheet: D1, D2, D3, D4, D5, D6, D7
Changed lines of the file:
@@
 	1    0    0    -1
 $EndComp
-$Comp
-L Device:LED D1
-U 1 1 61A1AB90
-P 4800 6050
-F 0 "D1" H 4793 5795 50  0000 C CNN
-F 1 "LED" H 4793 5886 50  0000 C CNN
-F 2 "LED_SMD:LED_0603_1608Metric_Castellated" H 4800 6050 50  0001 C CNN
-F 3 "~" H 4800 6050 50  0001 C CNN
-	1    4800 6050
-	-1   0    0    1
-$EndComp
-Wire Wire Line
-	4650 6450 4650 6350
-Wire Wire Line
-	5200 6450 5200 6350
-Wire Wire Line
-	5750 6450 5750 6350
-Wire Wire Line
-	5200 6050 5200 5950
-Wire Wire Line
-	4650 6050 4650 5950
-Wire Wire Line
-	5750 6050 5750 5950
-Wire Wire Line
-	4950 5800 4950 6050
-Connection ~ 4950 6050
-Wire Wire Line
-	4550 5950 4650 5950
-Connection ~ 4650 5950
-Connection ~ 5200 5950
-Wire Wire Line
-	5200 5950 5750 5950
-Connection ~ 5750 5950
-Connection ~ 4650 6350
-Connection ~ 5200 6350
-Wire Wire Line
-	5200 6350 5750 6350
-Connection ~ 5750 6350
-Text GLabel 4550 5950 3    50   Input ~ 0
-LED_A
-Text GLabel 4550 6350 3    50   Input ~ 0
-LED_B
-Wire Wire Line
-	4550 6350 4650 6350
-Text GLabel 6050 5800 2    50   Input ~ 0
-LED_3
-Text GLabel 5500 5800 2    50   Input ~ 0
-LED_2
-Text GLabel 4950 5800 2    50   Input ~ 0
-LED_1
 Connection ~ 3600 1250
 $Comp
@@
 	1    0    0    -1
 $EndComp
-Wire Wire Line
-	4650 5950 5200 5950
-Wire Wire Line
-	4650 6350 5200 6350
 $Comp
 L Connector:TestPoint TP2
@@
 	0    -1   -1   0
 $EndComp
-Text GLabel 7950 1550 2    50   Input ~ 0
-LED_2
-Text GLabel 7950 1450 2    50   Input ~ 0
-LED_1
-Text GLabel 7950 2550 2    50   Input ~ 0
-LED_B
 Text GLabel 7950 1650 2    50   Input ~ 0
 Up
@@
 L power:GND #PWR013
 U 1 1 61A23D2A
-P 7250 4950
-F 0 "#PWR013" H 7250 4700 50  0001 C CNN
-F 1 "GND" H 7255 4777 50  0000 C CNN
-F 2 "" H 7250 4950 50  0001 C CNN
-F 3 "" H 7250 4950 50  0001 C CNN
-	1    7250 4950
-	0    -1   1    0
+P 7150 4950
+F 0 "#PWR013" H 7150 4700 50  0001 C CNN
+F 1 "GND" H 7155 4777 50  0000 C CNN
+F 2 "" H 7150 4950 50  0001 C CNN
+F 3 "" H 7150 4950 50  0001 C CNN
+	1    7150 4950
+	0    1    -1   0
 $EndComp
 Wire Wire Line
@@
 Wire Wire Line
 	7150 4950 7250 4950
-Connection ~ 7250 4950
-Text GLabel 7950 2450 2    50   Input ~ 0
-LED_A
-Text GLabel 7950 2250 2    50   Input ~ 0
-LED_3
 $Comp
 L Connector:TestPoint TP11
@@
 	1    0    0    -1
 $EndComp
-Text GLabel 6600 5800 2    50   Input ~ 0
-LED_4
-Wire Wire Line
-	5750 6350 6300 6350
-Wire Wire Line
-	6300 6350 6300 6450
-Text GLabel 7950 2350 2    50   Input ~ 0
-LED_4
 Text GLabel 4200 3500 0    50   Input ~ 0
 Rmouse
@@
 Text GLabel 4650 2400 0    50   Input ~ 0
 8
-Wire Wire Line
-	4950 6050 4950 6450
-Wire Wire Line
-	6050 5800 6050 6050
-Wire Wire Line
-	5500 5800 5500 6050
-$Comp
-L Device:LED D2
-U 1 1 61AA2C14
-P 5350 6050
-F 0 "D2" H 5343 5795 50  0000 C CNN
-F 1 "LED" H 5343 5886 50  0000 C CNN
-F 2 "LED_SMD:LED_0603_1608Metric_Castellated" H 5350 6050 50  0001 C CNN
-F 3 "~" H 5350 6050 50  0001 C CNN
-	1    5350 6050
-	-1   0    0    1
-$EndComp
-Connection ~ 5500 6050
-Wire Wire Line
-	5500 6050 5500 6450
-$Comp
-L Device:LED D3
-U 1 1 61AA2FD4
-P 5900 6050
-F 0 "D3" H 5893 5795 50  0000 C CNN
-F 1 "LED" H 5893 5886 50  0000 C CNN
-F 2 "LED_SMD:LED_0603_1608Metric_Castellated" H 5900 6050 50  0001 C CNN
-F 3 "~" H 5900 6050 50  0001 C CNN
-	1    5900 6050
-	-1   0    0    1
-$EndComp
-Connection ~ 6050 6050
-Wire Wire Line
-	6050 6050 6050 6450
-$Comp
-L Device:LED D4
-U 1 1 61AA32CE
-P 6450 6450
-F 0 "D4" H 6443 6195 50  0000 C CNN
-F 1 "LED" H 6443 6286 50  0000 C CNN
-F 2 "LED_SMD:LED_0603_1608Metric_Castellated" H 6450 6450 50  0001 C CNN
-F 3 "~" H 6450 6450 50  0001 C CNN
-	1    6450 6450
-	-1   0    0    1
-$EndComp
-$Comp
-L Device:LED D7
-U 1 1 61AA3601
-P 5900 6450
-F 0 "D7" H 5893 6195 50  0000 C CNN
-F 1 "LED" H 5893 6286 50  0000 C CNN
-F 2 "LED_SMD:LED_0603_1608Metric_Castellated" H 5900 6450 50  0001 C CNN
-F 3 "~" H 5900 6450 50  0001 C CNN
-	1    5900 6450
-	-1   0    0    1
-$EndComp
-Connection ~ 6050 6450
-Wire Wire Line
-	6050 6450 6050 6650
-$Comp
-L Device:LED D6
-U 1 1 61AA3DB9
-P 5350 6450
-F 0 "D6" H 5343 6195 50  0000 C CNN
-F 1 "LED" H 5343 6286 50  0000 C CNN
-F 2 "LED_SMD:LED_0603_1608Metric_Castellated" H 5350 6450 50  0001 C CNN
-F 3 "~" H 5350 6450 50  0001 C CNN
-	1    5350 6450
-	-1   0    0    1
-$EndComp
-Connection ~ 5500 6450
-Wire Wire Line
-	5500 6450 5500 6650
-$Comp
-L Device:LED D5
-U 1 1 61AA408B
-P 4800 6450
-F 0 "D5" H 4793 6195 50  0000 C CNN
-F 1 "LED" H 4793 6286 50  0000 C CNN
-F 2 "LED_SMD:LED_0603_1608Metric_Castellated" H 4800 6450 50  0001 C CNN
-F 3 "~" H 4800 6450 50  0001 C CNN
-	1    4800 6450
-	-1   0    0    1
-$EndComp
-Connection ~ 4950 6450
-Wire Wire Line
-	4950 6450 4950 6650
 Text GLabel 2000 5050 2    50   Input ~ 0
 Enter
 Text GLabel 6550 1550 0    50   Input ~ 0
 Enter
-Connection ~ 6300 6350
-Wire Wire Line
-	6300 6350 6900 6350
-Connection ~ 6600 6450
-Wire Wire Line
-	6600 6450 6600 6650
-Wire Wire Line
-	5750 5950 6900 5950
-Wire Wire Line
-	6600 5800 6600 6450
 $Comp
 L Device:C C5
@@
 	10650 3950 10850 3950
 Connection ~ 10850 3950
+Connection ~ 7150 4950
+$Comp
+L Device:LED D5
+U 1 1 61AA408B
+P 8100 2650
+F 0 "D5" H 8093 2395 50  0000 C CNN
+F 1 "LED" H 8093 2486 50  0000 C CNN
+F 2 "LED_SMD:LED_0603_1608Metric_Castellated" H 8100 2650 50  0001 C CNN
+F 3 "~" H 8100 2650 50  0001 C CNN
+	1    8100 2650
+	-1   0    0    1
+$EndComp
+$Comp
+L Device:LED D6
+U 1 1 61AA3DB9
+P 8100 2750
+F 0 "D6" H 8093 2495 50  0000 C CNN
+F 1 "LED" H 8093 2586 50  0000 C CNN
+F 2 "LED_SMD:LED_0603_1608Metric_Castellated" H 8100 2750 50  0001 C CNN
+F 3 "~" H 8100 2750 50  0001 C CNN
+	1    8100 2750
+	-1   0    0    1
+$EndComp
+$Comp
+L Device:LED D7
+U 1 1 61AA3601
+P 8100 2850
+F 0 "D7" H 8093 2595 50  0000 C CNN
+F 1 "LED" H 8093 2686 50  0000 C CNN
+F 2 "LED_SMD:LED_0603_1608Metric_Castellated" H 8100 2850 50  0001 C CNN
+F 3 "~" H 8100 2850 50  0001 C CNN
+	1    8100 2850
+	-1   0    0    1
+$EndComp
+$Comp
+L Device:LED D4
+U 1 1 61AA32CE
+P 8100 2550
+F 0 "D4" H 8093 2295 50  0000 C CNN
+F 1 "LED" H 8093 2386 50  0000 C CNN
+F 2 "LED_SMD:LED_0603_1608Metric_Castellated" H 8100 2550 50  0001 C CNN
+F 3 "~" H 8100 2550 50  0001 C CNN
+	1    8100 2550
+	-1   0    0    1
+$EndComp
+Wire Wire Line
+	8250 2250 8250 2350
+Connection ~ 8250 2350
+Wire Wire Line
+	8250 2350 8250 2450
+Connection ~ 8250 2450
+Wire Wire Line
+	8250 2450 8250 2550
+Connection ~ 8250 2550
+Wire Wire Line
+	8250 2550 8250 2650
+Connection ~ 8250 2650
+Wire Wire Line
+	8250 2650 8250 2750
+Connection ~ 8250 2750
+Wire Wire Line
+	8250 2750 8250 2850
+Connection ~ 8250 2850
+$Comp
+L power:GND #PWR0101
+U 1 1 61C076C0
+P 8250 2850
+F 0 "#PWR0101" H 8250 2600 50  0001 C CNN
+F 1 "GND" H 8255 2677 50  0000 C CNN
+F 2 "" H 8250 2850 50  0001 C CNN
+F 3 "" H 8250 2850 50  0001 C CNN
+	1    8250 2850
+	1    0    0    -1
+$EndComp
+$Comp
+L Device:LED D3
+U 1 1 61AA2FD4
+P 8100 2450
+F 0 "D3" H 8093 2195 50  0000 C CNN
+F 1 "LED" H 8093 2286 50  0000 C CNN
+F 2 "LED_SMD:LED_0603_1608Metric_Castellated" H 8100 2450 50  0001 C CNN
+F 3 "~" H 8100 2450 50  0001 C CNN
+	1    8100 2450
+	-1   0    0    1
+$EndComp
+$Comp
+L Device:LED D2
+U 1 1 61AA2C14
+P 8100 2350
+F 0 "D2" H 8093 2095 50  0000 C CNN
+F 1 "LED" H 8093 2186 50  0000 C CNN
+F 2 "LED_SMD:LED_0603_1608Metric_Castellated" H 8100 2350 50  0001 C CNN
+F 3 "~" H 8100 2350 50  0001 C CNN
+	1    8100 2350
+	-1   0    0    1
+$EndComp
+$Comp
+L Device:LED D1
+U 1 1 61A1AB90
+P 8100 2250
+F 0 "D1" H 8093 1995 50  0000 C CNN
+F 1 "LED" H 8093 2086 50  0000 C CNN
+F 2 "LED_SMD:LED_0603_1608Metric_Castellated" H 8100 2250 50  0001 C CNN
+F 3 "~" H 8100 2250 50  0001 C CNN
+	1    8100 2250
+	-1   0    0    1
+$EndComp
 $EndSCHEMATC

Commit message: Updated Files
Parts:
- added C6, C7: C, Capacitor_SMD:C_0603_1608Metric_Pad1.08x0.95mm_HandSolder, symbol Device:C
- added Y1: Crystal, Crystal:Crystal_SMD_HC49-SD, symbol Device:Crystal
- J2, J3: footprint CapTouchKeyboard:8-pinheader -> Connector_PinSocket_2.54mm:PinSocket_1x08_P2.54mm_Vertical; symbol Cap-Touch-Controller:8-pin_header -> Connector:Conn_01x08_Female
Connections:
- net GND: now also C6.2, C7.1
- net at U1.1 (PA00): now also C6.1, Y1.1
- net at U1.2 (PA01): now also C7.2, Y1.2
Changed lines of the file:
@@
 F 3 "" H 2700 2450 50  0001 C CNN
 	1    2700 2450
-	0    -1   -1   0
+	1    0    0    -1
 $EndComp
 Connection ~ 2700 2450
@@
 	0    1    1    0
 $EndComp
-$Comp
-L power:GND #PWR03
-U 1 1 61A4F7DA
-P 7850 1150
-F 0 "#PWR03" H 7850 900 50  0001 C CNN
-F 1 "GND" V 7855 1022 50  0000 R CNN
-F 2 "" H 7850 1150 50  0001 C CNN
-F 3 "" H 7850 1150 50  0001 C CNN
-	1    7850 1150
-	0    -1   -1   0
-$EndComp
 Text GLabel 7950 1650 2    50   Input ~ 0
 Up
@@
 $EndComp
 Wire Wire Line
-	6950 1150 7050 1150
-$Comp
-L MCU_Microchip_SAMD:ATSAMD21J15B-A U1
-U 1 1 61A3E6B2
-P 7250 3050
-F 0 "U1" H 7250 1061 50  0000 C CNN
-F 1 "ATSAMD21J15B-A" H 7250 970 50  0000 C CNN
-F 2 "Package_QFP:TQFP-64_10x10mm_P0.5mm" H 8200 1200 50  0001 C CNN
-F 3 "http://ww1.microchip.com/downloads/en/DeviceDoc/SAM_D21_DA1_Family_Data%20Sheet_DS40001882E.pdf" H 7250 4050 50  0001 C CNN
-	1    7250 3050
-	-1   0    0    -1
-$EndComp
-Wire Wire Line
-	7250 1150 7350 1150
-Connection ~ 7350 1150
-Wire Wire Line
-	7050 1150 7150 1150
-Connection ~ 7050 1150
-Connection ~ 7250 1150
-Connection ~ 7150 1150
-Wire Wire Line
-	7150 1150 7250 1150
-Wire Wire Line
 	7150 4950 7250 4950
 $Comp
@@
 Rmouse
 $Comp
-L Cap-Touch-Controller:8-pin_header J3
+L Connector:Conn_01x08_Female J3
 U 1 1 61A89829
-P 1900 4700
-F 0 "J3" V 1025 4700 50  0000 C CNN
-F 1 "8-pin_header" V 1116 4700 50  0000 C CNN
-F 2 "CapTouchKeyboard:8-pinheader" H 1850 4900 60  0001 L CNN
-F 3 "" H 1850 5000 60  0001 L CNN
-	1    1900 4700
-	0    1    1    0
-$EndComp
-$Comp
-L Cap-Touch-Controller:8-pin_header J2
-U 1 1 61A8A194
-P 4750 2050
-F 0 "J2" V 4549 1908 50  0000 R CNN
-F 1 "8-pin_header" V 4640 1908 50  0000 R CNN
-F 2 "CapTouchKeyboard:8-pinheader" H 4700 2250 60  0001 L CNN
-F 3 "" H 4700 2350 60  0001 L CNN
-	1    4750 2050
-	0    -1   1    0
+P 1800 4650
+F 0 "J3" V 925 4650 50  0000 C CNN
+F 1 "8-pin_header" V 1016 4650 50  0000 C CNN
+F 2 "Connector_PinSocket_2.54mm:PinSocket_1x08_P2.54mm_Vertical" H 1750 4850 60  0001 L CNN
+F 3 "" H 1750 4950 60  0001 L CNN
+	1    1800 4650
+	-1   0    0    -1
 $EndComp
 Text GLabel 6550 1650 0    50   Input ~ 0
@@
 	10650 3950 10850 3950
 Connection ~ 10850 3950
-Connection ~ 7150 4950
 $Comp
 L Device:LED D5
@@
 	-1   0    0    1
 $EndComp
+$Comp
+L Device:C C7
+U 1 1 61C235C6
+P 8750 1650
+F 0 "C7" V 8498 1650 50  0000 C CNN
+F 1 "C" V 8589 1650 50  0000 C CNN
+F 2 "Capacitor_SMD:C_0603_1608Metric_Pad1.08x0.95mm_HandSolder" H 8788 1500 50  0001 C CNN
+F 3 "~" H 8750 1650 50  0001 C CNN
+	1    8750 1650
+	0    1    -1   0
+$EndComp
+Wire Wire Line
+	8900 1350 8900 1650
+$Comp
+L power:GND #PWR0102
+U 1 1 61C251BC
+P 8900 1650
+F 0 "#PWR0102" H 8900 1400 50  0001 C CNN
+F 1 "GND" H 8905 1477 50  0000 C CNN
+F 2 "" H 8900 1650 50  0001 C CNN
+F 3 "" H 8900 1650 50  0001 C CNN
+	1    8900 1650
+	-1   0    0    -1
+$EndComp
+Connection ~ 8900 1650
+$Comp
+L Device:C C6
+U 1 1 61C23035
+P 8750 1350
+F 0 "C6" V 8498 1350 50  0000 C CNN
+F 1 "C" V 8589 1350 50  0000 C CNN
+F 2 "Capacitor_SMD:C_0603_1608Metric_Pad1.08x0.95mm_HandSolder" H 8788 1200 50  0001 C CNN
+F 3 "~" H 8750 1350 50  0001 C CNN
+	1    8750 1350
+	0    -1   1    0
+$EndComp
+$Comp
+L Device:Crystal Y1
+U 1 1 61C222CD
+P 8600 1500
+F 0 "Y1" V 8554 1631 50  0000 L CNN
+F 1 "Crystal" V 8645 1631 50  0000 L CNN
+F 2 "Crystal:Crystal_SMD_HC49-SD" H 8600 1500 50  0001 C CNN
+F 3 "~" H 8600 1500 50  0001 C CNN
+	1    8600 1500
+	0    -1   1    0
+$EndComp
+Connection ~ 7150 4950
+Connection ~ 7150 1150
+Connection ~ 7250 1150
+Connection ~ 7050 1150
+Connection ~ 7350 1150
+Wire Wire Line
+	7150 1150 7250 1150
+Wire Wire Line
+	7250 1150 7350 1150
+Wire Wire Line
+	7050 1150 7150 1150
+Wire Wire Line
+	6950 1150 7050 1150
+$Comp
+L MCU_Microchip_SAMD:ATSAMD21J15B-A U1
+U 1 1 61A3E6B2
+P 7250 3050
+F 0 "U1" H 7250 1061 50  0000 C CNN
+F 1 "ATSAMD21J15B-A" H 7250 970 50  0000 C CNN
+F 2 "Package_QFP:TQFP-64_10x10mm_P0.5mm" H 8200 1200 50  0001 C CNN
+F 3 "http://ww1.microchip.com/downloads/en/DeviceDoc/SAM_D21_DA1_Family_Data%20Sheet_DS40001882E.pdf" H 7250 4050 50  0001 C CNN
+	1    7250 3050
+	-1   0    0    -1
+$EndComp
+Wire Wire Line
+	7950 1550 8200 1550
+Wire Wire Line
+	8200 1550 8200 1650
+Wire Wire Line
+	8200 1650 8600 1650
+Connection ~ 8600 1650
+Wire Wire Line
+	8600 1350 7950 1350
+Wire Wire Line
+	7950 1350 7950 1450
+Connection ~ 8600 1350
+$Comp
+L power:GND #PWR03
+U 1 1 61A4F7DA
+P 7850 1150
+F 0 "#PWR03" H 7850 900 50  0001 C CNN
+F 1 "GND" V 7855 1022 50  0000 R CNN
+F 2 "" H 7850 1150 50  0001 C CNN
+F 3 "" H 7850 1150 50  0001 C CNN
+	1    7850 1150
+	0    -1   -1   0
+$EndComp
+$Comp
+L Connector:Conn_01x08_Female J2
+U 1 1 61A8A194
+P 4850 2000
+F 0 "J2" V 4649 1858 50  0000 R CNN
+F 1 "8-pin_header" V 4740 1858 50  0000 R CNN
+F 2 "Connector_PinSocket_2.54mm:PinSocket_1x08_P2.54mm_Vertical" H 4800 2200 60  0001 L CNN
+F 3 "" H 4800 2300 60  0001 L CNN
+	1    4850 2000
+	1    0    0    -1
+$EndComp
 $EndSCHEMATC

Commit message: New files
Parts:
- removed TP10, TP9: TestPoint, CapTouchKeyboard:PC_TEST_POINT_SMD, symbol Connector:TestPoint
- added SW1: SW_Push, Button_Switch_SMD:SW_Push_1P1T_NO_6x6mm_H9.5mm, symbol Switch:SW_Push
Connections:
- net GND: now also SW1.1
- net ~RST: now also SW1.2
Changed lines of the file:
@@
 	-1   0    0    1
 $EndComp
-Text GLabel 9250 5300 3    50   Input ~ 0
+Text GLabel 9150 5300 3    50   Input ~ 0
 ~RST
-$Comp
-L Connector:TestPoint TP10
-U 1 1 61A15B4A
-P 9250 5300
-F 0 "TP10" H 9308 5418 50  0000 L CNN
-F 1 "TestPoint" H 9308 5327 50  0000 L CNN
-F 2 "CapTouchKeyboard:PC_TEST_POINT_SMD" H 9450 5300 50  0001 C CNN
-F 3 "~" H 9450 5300 50  0001 C CNN
-	1    9250 5300
-	1    0    0    -1
-$EndComp
 Connection ~ 3600 1250
-$Comp
-L Connector:TestPoint TP9
-U 1 1 61A4565D
-P 8750 5300
-F 0 "TP9" H 8808 5418 50  0000 L CNN
-F 1 "TestPoint" H 8808 5327 50  0000 L CNN
-F 2 "CapTouchKeyboard:PC_TEST_POINT_SMD" H 8950 5300 50  0001 C CNN
-F 3 "~" H 8950 5300 50  0001 C CNN
-	1    8750 5300
-	1    0    0    -1
-$EndComp
 $Comp
 L power:GND #PWR014
@@
 	1    0    0    -1
 $EndComp
+$Comp
+L Switch:SW_Push SW1
+U 1 1 61C63258
+P 8950 5300
+F 0 "SW1" H 8950 5585 50  0000 C CNN
+F 1 "SW_Push" H 8950 5494 50  0000 C CNN
+F 2 "Button_Switch_SMD:SW_Push_1P1T_NO_6x6mm_H9.5mm" H 8950 5600 50  0001 C CNN
+F 3 "http://www.apem.com/int/index.php?controller=attachment&id_attachment=1371" H 8950 5600 50  0001 C CNN
+	1    8950 5300
+	1    0    0    -1
+$EndComp
