File: kicad-files/Cap Touch Controller.kicad_pcb (KiCad board)
At the start: 2 copper layers, 28 parts, among them J1 USB_C_Receptacle_USB2.0, J2 8-pin_header, J3 8-pin_header, U1 ATSAMD21J15B-A, U2 MIC5365-2.8YC5

Commit message: New Files
Parts:
- moved R2 0.67 mm to (40.5, 36.0)
- moved C4 0.44 mm to (74.5, 40.0)
- moved C2 0.37 mm to (73.0, 40.0)
- moved C5 0.36 mm to (71.5, 40.0)
- moved R1 0.32 mm to (35.5, 36.0)
- moved U1 0.27 mm to (63.0, 41.0)
- moved U2 0.25 mm to (37.5, 40.0)
- moved C3 0.23 mm to (35.0, 40.0)
- moved C1 0.12 mm to (66.0, 32.5)
Connections:
- D1 pad 1: LED_1 -> GND
- D1 pad 2: LED_A -> Net-(D1-Pad2)
- D2 pad 1: LED_2 -> GND
- D2 pad 2: LED_A -> Net-(D2-Pad2)
- D3 pad 1: LED_3 -> GND
- D3 pad 2: LED_A -> Net-(D3-Pad2)
- D4 pad 1: LED_4 -> GND
- D4 pad 2: LED_B -> Net-(D4-Pad2)
- D5 pad 1: LED_1 -> GND
- D5 pad 2: LED_B -> Net-(D5-Pad2)
- D6 pad 1: LED_2 -> GND
- D6 pad 2: LED_B -> Net-(D6-Pad2)
- D7 pad 1: LED_3 -> GND
- D7 pad 2: LED_B -> Net-(D7-Pad2)
- U1 pad 1: LED_1 -> Net-(U1-Pad1)
- U1 pad 17: LED_3 -> Net-(D1-Pad2)
- U1 pad 18: LED_4 -> Net-(D2-Pad2)
- U1 pad 19: LED_A -> Net-(D3-Pad2)
- U1 pad 2: LED_2 -> Net-(U1-Pad2)
- U1 pad 20: LED_B -> Net-(D4-Pad2)
- U1 pad 29: Net-(U1-Pad29) -> Net-(D5-Pad2)
- U1 pad 30: Net-(U1-Pad30) -> Net-(D6-Pad2)
- U1 pad 31: Net-(U1-Pad31) -> Net-(D7-Pad2)
Routing:
- net GND: track 102.8 -> 249.3 mm, vias 0 -> 1
- net LED_B: track 106.3 -> 0.00 mm, vias 1 -> 0
- net LED_1: track 69.3 -> 0.00 mm, vias 1 -> 0
- net LED_A: track 69.0 -> 0.00 mm, vias 1 -> 0
- net LED_3: track 60.8 -> 0.00 mm, vias 1 -> 0
- net Net-(D4-Pad2): track 0.00 -> 49.9 mm, vias 0 -> 1
- net Net-(D7-Pad2): track 0.00 -> 46.0 mm, vias 0 -> 1
- net Down: track 129.3 -> 86.0 mm
- net LED_4: track 42.3 -> 0.00 mm, vias 1 -> 0
- net Net-(D3-Pad2): track 0.00 -> 41.5 mm, vias 0 -> 1
- net LED_2: track 38.2 -> 0.00 mm, vias 1 -> 0
- net Net-(D5-Pad2): track 0.00 -> 32.6 mm, vias 0 -> 1
- net Net-(D1-Pad2): track 0.00 -> 25.2 mm, vias 0 -> 1
- net Net-(D2-Pad2): track 0.00 -> 23.7 mm, vias 0 -> 1
- net Net-(D6-Pad2): track 0.00 -> 20.8 mm, vias 0 -> 1
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Other:
- board outline added: 92.4 x 53 mm

Commit message: Updated Files
Parts:
- added C6: C, Capacitor_SMD:C_0603_1608Metric_Pad1.08x0.95mm_HandSolder, B.Cu at (93.1, 40.0)
- added C7: C, Capacitor_SMD:C_0603_1608Metric_Pad1.08x0.95mm_HandSolder, B.Cu at (76.8, 40.0)
- added Y1: Crystal, Crystal:Crystal_SMD_HC49-SD, B.Cu at (84.5, 40.0)
- J2, J3: footprint CapTouchKeyboard:8-pinheader -> Connector_PinSocket_2.54mm:PinSocket_1x08_P2.54mm_Vertical
- moved J2 8.89 mm to (114.8, 29.1), turned to 180 degrees
- moved J3 8.89 mm to (28.4, 29.1), turned to 180 degrees
Routing:
- net Net-(C6-Pad1): track 0.00 -> 24.8 mm, vias 0 -> 2
- net Net-(C7-Pad2): track 0.00 -> 16.4 mm, vias 0 -> 2
- net GND: track 249.3 -> 263.7 mm, vias 1 -> 2

Commit message: New files
Parts:
- removed TP10, TP9: TestPoint, CapTouchKeyboard:PC_TEST_POINT_SMD
- added SW1: SW_Push, Button_Switch_SMD:SW_Push_1P1T_NO_6x6mm_H9.5mm, B.Cu at (58.0, 31.0)
Connections:
- net +3V3 renamed +2V8
- net +5V renamed VBUS
Routing:
- net Rmouse: track 90.5 -> 112.1 mm, vias 1 -> 0
- net ~RST: track 3.82 -> 14.7 mm
- net GND: track 263.7 -> 273.7 mm, vias 2 -> 1
- net Net-(D4-Pad2): track 49.9 -> 43.2 mm
- net Right: track 65.6 -> 59.1 mm
- net MouseClick: track 91.9 -> 95.1 mm
- net Net-(C7-Pad2): track 16.4 -> 14.4 mm, vias 2 -> 0
- net VBUS: track 15.9 -> 17.5 mm
- net Up: track 59.9 -> 58.5 mm
- net Down: track 86.0 -> 84.9 mm
- net +2V8: track 59.7 -> 60.8 mm
- net Left: track 76.7 -> 77.7 mm
- net Net-(C6-Pad1): track 24.8 -> 25.5 mm, vias 2 -> 0
- net Net-(D5-Pad2): track 32.6 -> 33.2 mm
- net Enter: vias 0 -> 1
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
Commit message: KiCad 6 files
Parts:
- removed C6, C7: C, Capacitor_SMD:C_0603_1608Metric_Pad1.08x0.95mm_HandSolder
- removed Y1: Crystal, Crystal:Crystal_SMD_HC49-SD
- added R3: 1k, Resistor_SMD:R_0603_1608Metric_Pad0.98x0.95mm_HandSolder, B.Cu at (50.0, 28.4)
- added R4: 1k, Resistor_SMD:R_0603_1608Metric_Pad0.98x0.95mm_HandSolder, B.Cu at (88.0, 43.0)
- added R5: 1k, Resistor_SMD:R_0603_1608Metric_Pad0.98x0.95mm_HandSolder, B.Cu at (106.0, 43.0)
- added R6: 1k, Resistor_SMD:R_0603_1608Metric_Pad0.98x0.95mm_HandSolder, B.Cu at (28.4, 52.5)
- added R7: 1k, Resistor_SMD:R_0603_1608Metric_Pad0.98x0.95mm_HandSolder, B.Cu at (50.0, 75.4)
- added R8: 1k, Resistor_SMD:R_0603_1608Metric_Pad0.98x0.95mm_HandSolder, B.Cu at (75.4, 50.5)
- added R9: 1k, Resistor_SMD:R_0603_1608Metric_Pad0.98x0.95mm_HandSolder, B.Cu at (97.0, 63.0)
- added TP7: TestPoint, TestPoint:TestPoint_Pad_D1.0mm, B.Cu at (66.5, 29.1)
- added TP8: TestPoint, TestPoint:TestPoint_Pad_D1.0mm, B.Cu at (71.6, 34.2)
- added TP9: TestPoint, TestPoint:TestPoint_Pad_D1.0mm, B.Cu at (69.0, 34.2)
- D1, D2, D3, D4, D5, D6, D7: footprint LED_SMD:LED_0603_1608Metric_Castellated -> LED_SMD:LED_0603_1608Metric_Pad1.05x0.95mm_HandSolder
- U2: value MIC5365-2.8YC5 -> MIC5365-3.3YD5; footprint Package_TO_SOT_SMD:SOT-353_SC-70-5 -> Package_TO_SOT_SMD:SOT-23-5
- moved C1 2.00 mm to (64.0, 32.5)
- moved D1 0.80 mm to (52.0, 28.4)
- moved C2 0.50 mm to (73.0, 39.5)
- moved C4 0.50 mm to (74.5, 39.5)
- moved C5 0.50 mm to (71.5, 39.5)
- turned D2 to 180 degrees
Connections:
- net +2V8 renamed +3V3
- net Net-(U1-Pad35) renamed SDA
- net Net-(U1-Pad36) renamed SCL
- net ~RST renamed ~{RST}
- D1 pad 1: GND -> Net-(D1-Pad1)
- D2 pad 1: GND -> Net-(D2-Pad1)
- D3 pad 1: GND -> Net-(D3-Pad1)
- D4 pad 1: GND -> Net-(D4-Pad1)
- D5 pad 1: GND -> Net-(D5-Pad1)
- D6 pad 1: GND -> Net-(D6-Pad1)
- D7 pad 1: GND -> Net-(D7-Pad1)
- J1 pad A8: Net-(J1-PadA8) -> unconnected-(J1-PadA8)
- J1 pad B8: Net-(J1-PadB8) -> unconnected-(J1-PadB8)
- U1 pad 1: Net-(C6-Pad1) -> unconnected-(U1-Pad1)
- U1 pad 2: Net-(C7-Pad2) -> unconnected-(U1-Pad2)
- U1 pad 23: Net-(U1-Pad23) -> unconnected-(U1-Pad23)
- U1 pad 24: Net-(U1-Pad24) -> unconnected-(U1-Pad24)
- U1 pad 25: Net-(U1-Pad25) -> unconnected-(U1-Pad25)
- U1 pad 26: Net-(U1-Pad26) -> unconnected-(U1-Pad26)
- U1 pad 27: Net-(U1-Pad27) -> unconnected-(U1-Pad27)
- U1 pad 28: Net-(U1-Pad28) -> unconnected-(U1-Pad28)
- U1 pad 32: Net-(U1-Pad32) -> unconnected-(U1-Pad32)
- U1 pad 37: Net-(U1-Pad37) -> unconnected-(U1-Pad37)
- U1 pad 38: Net-(U1-Pad38) -> unconnected-(U1-Pad38)
- U1 pad 39: Net-(U1-Pad39) -> unconnected-(U1-Pad39)
- U1 pad 40: Net-(U1-Pad40) -> unconnected-(U1-Pad40)
- U1 pad 41: Net-(U1-Pad41) -> unconnected-(U1-Pad41)
- U1 pad 42: Net-(U1-Pad42) -> unconnected-(U1-Pad42)
- U1 pad 43: Net-(U1-Pad43) -> unconnected-(U1-Pad43)
- U1 pad 44: Net-(U1-Pad44) -> unconnected-(U1-Pad44)
- U1 pad 49: Net-(U1-Pad49) -> unconnected-(U1-Pad49)
- U1 pad 50: Net-(U1-Pad50) -> unconnected-(U1-Pad50)
- U1 pad 51: Net-(U1-Pad51) -> unconnected-(U1-Pad51)
- U1 pad 53: Net-(U1-Pad53) -> unconnected-(U1-Pad53)
- U1 pad 57: Net-(U1-Pad57) -> SWCLK
- U1 pad 58: Net-(U1-Pad58) -> SWDIO
- U1 pad 59: Net-(U1-Pad59) -> unconnected-(U1-Pad59)
- U1 pad 60: Net-(U1-Pad60) -> unconnected-(U1-Pad60)
- U2 pad 4: Net-(U2-Pad4) -> unconnected-(U2-Pad4)
Routing:
- net GND: track 273.7 -> 20.1 mm, vias 1 -> 23
- net +3V3: track 60.8 -> 97.0 mm, vias 2 -> 0
- net Net-(C6-Pad1): track 25.5 -> 0.00 mm
- net Net-(C7-Pad2): track 14.4 -> 0.00 mm
- net Enter: track 46.0 -> 58.2 mm, vias 1 -> 0
- net SWCLK: track 0.00 -> 10.4 mm
- net Spacebar: track 145.8 -> 136.7 mm, vias 0 -> 1
- net SWDIO: track 0.00 -> 7.00 mm
- net Net-(D4-Pad2): track 43.2 -> 49.9 mm
- net Down: track 84.9 -> 91.4 mm
- net Net-(D6-Pad2): track 20.5 -> 26.9 mm
- net ~{RST}: track 14.7 -> 20.4 mm, vias 0 -> 2
- net Left: track 77.7 -> 83.0 mm
- net MouseClick: track 95.1 -> 90.0 mm
- net Right: track 59.1 -> 63.8 mm
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- added copper zone on B.Cu, net GND
- added copper zone on F.Cu, net GND
Other:
- net class Default removed

Commit message: Added Files
Parts:
- added J4: Conn_01x04_Female, Connector_JST:JST_SH_BM04B-SRSS-TB_1x04-1MP_P1.00mm_Vertical, B.Cu at (70.5, 28.0)
- R3, R4, R5, R6, R7, R8, R9: value 1k -> 100
- SW1: footprint Button_Switch_SMD:SW_Push_1P1T_NO_6x6mm_H9.5mm -> Button_Switch_SMD:SW_SPST_PTS645
- U1: value ATSAMD21J15B-A -> ATSAMD21J18A-A
- moved C2 31.5 mm to (41.5, 40.0)
- moved C4 31.5 mm to (43.0, 40.0)
- moved C5 31.5 mm to (40.0, 40.0)
- moved SW1 21.5 mm to (79.5, 30.4)
- moved C1 4.61 mm to (68.5, 33.5), turned to 135 degrees
- moved TP9 3.59 mm to (71.6, 36.7)
- moved TP7 2.54 mm to (66.5, 31.6)
- moved U1 1.50 mm to (63.0, 39.5), turned to 135 degrees
- moved D7 0.50 mm to (95.0, 62.5)
- moved R9 0.50 mm to (97.0, 62.5)
- turned D4 to 90 degrees
- turned R6 to 90 degrees
Connections:
- U1 pad 1: unconnected-(U1-Pad1) -> Net-(D3-Pad2)
- U1 pad 15: Rmouse -> MouseClick
- U1 pad 16: MouseClick -> Rmouse
- U1 pad 17: Net-(D1-Pad2) -> unconnected-(U1-Pad17)
- U1 pad 18: Net-(D2-Pad2) -> unconnected-(U1-Pad18)
- U1 pad 19: Net-(D3-Pad2) -> unconnected-(U1-Pad19)
- U1 pad 2: unconnected-(U1-Pad2) -> Net-(D2-Pad2)
- U1 pad 31: Net-(D7-Pad2) -> unconnected-(U1-Pad31)
- U1 pad 49: unconnected-(U1-Pad49) -> Net-(D1-Pad2)
- U1 pad 60: unconnected-(U1-Pad60) -> Net-(D7-Pad2)
Routing:
- net Spacebar: track 136.7 -> 106.6 mm
- net GND: track 20.1 -> 48.0 mm, vias 23 -> 17
- net Left: track 83.0 -> 57.8 mm
- net SDA: track 0.00 -> 16.9 mm
- net SCL: track 0.00 -> 15.2 mm
- net Net-(D4-Pad2): track 49.9 -> 38.8 mm
- net Net-(D1-Pad2): track 24.0 -> 14.0 mm
- net Enter: track 58.2 -> 48.3 mm, vias 0 -> 1
- net Rmouse: track 111.5 -> 102.0 mm
- net Net-(D3-Pad2): track 41.5 -> 36.1 mm
- net SWCLK: track 10.4 -> 5.01 mm
- net Net-(D2-Pad2): track 21.6 -> 16.6 mm
- net 6: track 46.1 -> 49.7 mm
- net Net-(D6-Pad2): track 26.9 -> 23.7 mm
- net 5: track 47.1 -> 50.3 mm
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
Commit message: Changed files
Parts:
- J4: footprint Connector_JST:JST_SH_BM04B-SRSS-TB_1x04-1MP_P1.00mm_Vertical -> Connector_JST:JST_SH_SM04B-SRSS-TB_1x04-1MP_P1.00mm_Horizontal
- moved R8 3.34 mm to (75.4, 53.8), turned to -90 degrees
- moved J4 0.50 mm to (70.5, 28.5), turned to 0 degrees
- turned D6 to 90 degrees
Connections:
- D6 pad 2: Net-(D6-Pad2) -> Net-(U1-Pad19)
- U1 pad 19: unconnected-(U1-Pad19) -> Net-(U1-Pad19)
- U1 pad 30: Net-(D6-Pad2) -> unconnected-(U1-Pad30)
Routing:
- net Net-(D6-Pad2): track 23.7 -> 0.00 mm, vias 1 -> 0
- net Net-(U1-Pad19): track 0.00 -> 19.3 mm, vias 0 -> 1
- net GND: track 48.0 -> 36.4 mm, vias 17 -> 18
- net SCL: track 15.2 -> 20.0 mm, vias 0 -> 2
- net SDA: track 16.9 -> 19.0 mm
- net +3V3: track 99.7 -> 98.0 mm
- net ~{RST}: track 21.1 -> 22.2 mm
